File: communication.sch (KiCad schematic (older format))
At the start: 17 parts, among them J5 Conn_01x03_Male, SW3 RESET, SW4 BOOT, U5 TJA1051T-3, U6 ESP32-WROOM-32

Commit message: fixed schematics error
Parts:
- C13: symbol prius_gen2-rescue:C_Small-Device -> prius_gen2-rescue:C_Small-Device-prius_gen2-rescue
- C30, C31, C32, C33: symbol prius_gen2-rescue:C-Device -> prius_gen2-rescue:C-Device-prius_gen2-rescue
- D2: symbol prius_gen2-rescue:D_TVS_x2_AAC-Device -> prius_gen2-rescue:D_TVS_x2_AAC-Device-prius_gen2-rescue
- D3: symbol prius_gen2-rescue:LED-Device -> prius_gen2-rescue:LED-Device-prius_gen2-rescue
- J5: symbol prius_gen2-rescue:Conn_01x03_Male-Connector -> prius_gen2-rescue:Conn_01x03_Male-Connector-prius_gen2-rescue
- JP1: symbol prius_gen2-rescue:SolderJumper_2_Open-Jumper -> prius_gen2-rescue:SolderJumper_2_Open-Jumper-prius_gen2-rescue
- R33, R34, R35, R36: symbol prius_gen2-rescue:R-Device -> prius_gen2-rescue:R-Device-prius_gen2-rescue
- SW3, SW4: symbol prius_gen2-rescue:SW_Push-Switch -> prius_gen2-rescue:SW_Push-Switch-prius_gen2-rescue
- U5: symbol prius_gen2-rescue:TJA1051T-3-Interface_CAN_LIN -> prius_gen2-rescue:TJA1051T-3-Interface_CAN_LIN-prius_gen2-rescue
- U6: symbol prius_gen2-rescue:ESP32-WROOM-32-RF_Module -> prius_gen2-rescue:ESP32-WROOM-32-RF_Module-prius_gen2-rescue
Changed lines of the file:
@@
 $EndDescr
 $Comp
-L prius_gen2-rescue:R-Device R33
+L prius_gen2-rescue:R-Device-prius_gen2-rescue R33
 U 1 1 60EC4A3C
 P 2685 3355
@@
 $EndComp
 $Comp
-L prius_gen2-rescue:SolderJumper_2_Open-Jumper JP1
+L prius_gen2-rescue:SolderJumper_2_Open-Jumper-prius_gen2-rescue JP1
 U 1 1 60EC5424
 P 3235 3355
@@
 	3085 3355 2835 3355
 $Comp
-L prius_gen2-rescue:+3V3-power #PWR0146
+L prius_gen2-rescue:+3V3-power-prius_gen2-rescue #PWR0146
 U 1 1 60EC75CC
 P 1975 4550
@@
 $EndComp
 $Comp
-L prius_gen2-rescue:ESP32-WROOM-32-RF_Module U6
+L prius_gen2-rescue:ESP32-WROOM-32-RF_Module-prius_gen2-rescue U6
 U 1 1 60EC899D
 P 7475 3825
@@
 $EndComp
 $Comp
-L prius_gen2-rescue:GND-power #PWR0147
+L prius_gen2-rescue:GND-power-prius_gen2-rescue #PWR0147
 U 1 1 60EC93A4
 P 7475 5325
@@
 	7475 5325 7475 5225
 $Comp
-L prius_gen2-rescue:+3V3-power #PWR0148
+L prius_gen2-rescue:+3V3-power-prius_gen2-rescue #PWR0148
 U 1 1 60ECA1BD
 P 8250 1925
@@
 	8325 2925 8075 2925
 $Comp
-L prius_gen2-rescue:TJA1051T-3-Interface_CAN_LIN U5
+L prius_gen2-rescue:TJA1051T-3-Interface_CAN_LIN-prius_gen2-rescue U5
 U 1 1 60FE982B
 P 2675 4450
@@
 $EndComp
 $Comp
-L prius_gen2-rescue:+5V-power #PWR0149
+L prius_gen2-rescue:+5V-power-prius_gen2-rescue #PWR0149
 U 1 1 60FEBEE7
 P 2675 3675
@@
 	1975 4550 2175 4550
 $Comp
-L prius_gen2-rescue:GND-power #PWR0150
+L prius_gen2-rescue:GND-power-prius_gen2-rescue #PWR0150
 U 1 1 60FF6A42
 P 2050 4750
@@
 	2050 4650 2175 4650
 $Comp
-L prius_gen2-rescue:GND-power #PWR0151
+L prius_gen2-rescue:GND-power-prius_gen2-rescue #PWR0151
 U 1 1 60FF73C6
 P 2675 4975
@@
 	2675 4975 2675 4850
 $Comp
-L prius_gen2-rescue:D_TVS_x2_AAC-Device D2
+L prius_gen2-rescue:D_TVS_x2_AAC-Device-prius_gen2-rescue D2
 U 1 1 60FFAE8A
 P 3825 4425
@@
 	3825 4025 4200 4025
 $Comp
-L prius_gen2-rescue:GND-power #PWR0152
+L prius_gen2-rescue:GND-power-prius_gen2-rescue #PWR0152
 U 1 1 60FFFD04
 P 4100 4425
@@
 CANL
 $Comp
-L prius_gen2-rescue:SW_Push-Switch SW3
+L prius_gen2-rescue:SW_Push-Switch-prius_gen2-rescue SW3
 U 1 1 6186DAB9
 P 6325 2850
@@
 NoConn ~ 8075 4925
 $Comp
-L prius_gen2-rescue:C-Device C31
+L prius_gen2-rescue:C-Device-prius_gen2-rescue C31
 U 1 1 6187C509
 P 7675 2125
@@
 $EndComp
 $Comp
-L prius_gen2-rescue:C-Device C32
+L prius_gen2-rescue:C-Device-prius_gen2-rescue C32
 U 1 1 6187C996
 P 8000 2125
@@
 $EndComp
 $Comp
-L prius_gen2-rescue:GND-power #PWR0153
+L prius_gen2-rescue:GND-power-prius_gen2-rescue #PWR0153
 U 1 1 6187CE43
 P 8200 2350
@@
 Connection ~ 7675 1925
 $Comp
-L prius_gen2-rescue:R-Device R36
+L prius_gen2-rescue:R-Device-prius_gen2-rescue R36
 U 1 1 618806A0
 P 8475 2100
@@
 	8075 2625 8475 2625
 $Comp
-L prius_gen2-rescue:C-Device C33
+L prius_gen2-rescue:C-Device-prius_gen2-rescue C33
 U 1 1 61881D8E
 P 8775 2500
@@
 $EndComp
 $Comp
-L prius_gen2-rescue:GND-power #PWR0154
+L prius_gen2-rescue:GND-power-prius_gen2-rescue #PWR0154
 U 1 1 61882C39
 P 8975 2750
@@
 Connection ~ 8775 2250
 $Comp
-L prius_gen2-rescue:SW_Push-Switch SW4
+L prius_gen2-rescue:SW_Push-Switch-prius_gen2-rescue SW4
 U 1 1 61882E01
 P 9200 2450
@@
 $EndComp
 $Comp
-L prius_gen2-rescue:LED-Device D3
+L prius_gen2-rescue:LED-Device-prius_gen2-rescue D3
 U 1 1 6188DBD9
 P 8675 3325
@@
 $EndComp
 $Comp
-L prius_gen2-rescue:R-Device R35
+L prius_gen2-rescue:R-Device-prius_gen2-rescue R35
 U 1 1 6188EDBA
 P 8350 3325
@@
 $EndComp
 $Comp
-L prius_gen2-rescue:GND-power #PWR0155
+L prius_gen2-rescue:GND-power-prius_gen2-rescue #PWR0155
 U 1 1 6188F393
 P 9050 3400
@@
 	8200 3325 8075 3325
 $Comp
-L prius_gen2-rescue:R-Device R34
+L prius_gen2-rescue:R-Device-prius_gen2-rescue R34
 U 1 1 61891C81
 P 6475 2400
@@
 $EndComp
 $Comp
-L prius_gen2-rescue:+3.3V-power #PWR0156
+L prius_gen2-rescue:+3.3V-power-prius_gen2-rescue #PWR0156
 U 1 1 618920DE
 P 6475 2175
@@
 $EndComp
 $Comp
-L prius_gen2-rescue:C-Device C30
+L prius_gen2-rescue:C-Device-prius_gen2-rescue C30
 U 1 1 618924A7
 P 6075 2850
@@
 $EndComp
 $Comp
-L prius_gen2-rescue:GND-power #PWR0157
+L prius_gen2-rescue:GND-power-prius_gen2-rescue #PWR0157
 U 1 1 618929D1
 P 6200 3200
@@
 	6475 2625 6875 2625
 $Comp
-L prius_gen2-rescue:Conn_01x03_Male-Connector J5
+L prius_gen2-rescue:Conn_01x03_Male-Connector-prius_gen2-rescue J5
 U 1 1 618C86EF
 P 8750 5025
@@
 $EndComp
 $Comp
-L prius_gen2-rescue:GND-power #PWR0158
+L prius_gen2-rescue:GND-power-prius_gen2-rescue #PWR0158
 U 1 1 618C8929
 P 9200 5275
@@
 	8075 3625 8250 3625
 $Comp
-L prius_gen2-rescue:C_Small-Device C?
+L prius_gen2-rescue:C_Small-Device-prius_gen2-rescue C?
 U 1 1 61D98C2A
 P 2850 3825
@@
 	2675 3725 2675 4050
 $Comp
-L prius_gen2-rescue:GND-power #PWR0188
+L prius_gen2-rescue:GND-power-prius_gen2-rescue #PWR0188
 U 1 1 61DA32D9
 P 2850 3950
