File: connectors.sch (KiCad schematic (older format))
At the start: 10 parts, among them J3 Conn_01x23, J4 Conn_01x14, U3 ULN2003A

Commit message: fixed schematics error
Parts:
- C18, C19: symbol prius_gen2-rescue:C-Device -> prius_gen2-rescue:C-Device-prius_gen2-rescue
- J3: symbol prius_gen2-rescue:Conn_01x23-Connector_Generic -> prius_gen2-rescue:Conn_01x23-Connector_Generic-prius_gen2-rescue
- J4: symbol prius_gen2-rescue:Conn_01x14-Connector_Generic -> prius_gen2-rescue:Conn_01x14-Connector_Generic-prius_gen2-rescue
- R22, R23, R24, R25, R26: symbol prius_gen2-rescue:R-Device -> prius_gen2-rescue:R-Device-prius_gen2-rescue
- U3: symbol prius_gen2-rescue:ULN2003A-Transistor_Array -> prius_gen2-rescue:ULN2003A-Transistor_Array-prius_gen2-rescue
Connections:
- net GND: no longer C18.1, J3.2 (Pin_2), R22.2, R23.2
- new net: C18.1, J3.2 (Pin_2), R22.2, R23.2
Changed lines of the file:
@@
 $EndDescr
 $Comp
-L prius_gen2-rescue:GND-power #PWR?
+L prius_gen2-rescue:GND-power-prius_gen2-rescue #PWR?
 U 1 1 611D14C9
 P 3700 5680
@@
 $EndComp
 $Comp
-L prius_gen2-rescue:+12V-power #PWR?
+L prius_gen2-rescue:+12V-power-prius_gen2-rescue #PWR?
 U 1 1 611D14DA
 P 3725 5225
@@
 $EndComp
 $Comp
-L prius_gen2-rescue:R-Device R?
+L prius_gen2-rescue:R-Device-prius_gen2-rescue R?
 U 1 1 611D14EF
 P 2800 2125
@@
 $EndComp
 $Comp
-L prius_gen2-rescue:GND-power #PWR?
+L prius_gen2-rescue:GND-power-prius_gen2-rescue #PWR?
 U 1 1 611D14F6
 P 3200 3125
@@
 $EndComp
 $Comp
-L prius_gen2-rescue:R-Device R?
+L prius_gen2-rescue:R-Device-prius_gen2-rescue R?
 U 1 1 611D14FC
 P 3550 2825
@@
 $EndComp
 $Comp
-L prius_gen2-rescue:C-Device C?
+L prius_gen2-rescue:C-Device-prius_gen2-rescue C?
 U 1 1 611D1502
 P 3200 2825
@@
 	1    0    0    -1
 $EndComp
-Wire Wire Line
-	3825 2625 3550 2625
 Connection ~ 2800 2625
 Wire Wire Line
 	2800 2625 2800 2275
 $Comp
-L prius_gen2-rescue:+5V-power #PWR?
+L prius_gen2-rescue:+5V-power-prius_gen2-rescue #PWR?
 U 1 1 611D150B
 P 2800 1850
@@
 Wire Wire Line
 	3200 3025 3550 3025
-Wire Wire Line
-	3825 2625 3825 3025
 Connection ~ 3200 3025
 Wire Wire Line
@@
 Wire Wire Line
 	3550 2675 3550 2625
-Connection ~ 3550 3025
-Wire Wire Line
-	3550 3025 3825 3025
-Connection ~ 3550 2625
 Wire Wire Line
 	3550 2625 3200 2625
@@
 	3200 2625 2800 2625
 $Comp
-L prius_gen2-rescue:+5V-power #PWR?
+L prius_gen2-rescue:+5V-power-prius_gen2-rescue #PWR?
 U 1 1 611D1521
 P 3750 3825
@@
 MIVT
 $Comp
-L prius_gen2-rescue:ULN2003A-Transistor_Array U3
+L prius_gen2-rescue:ULN2003A-Transistor_Array-prius_gen2-rescue U3
 U 1 1 6120D8B4
 P 7150 4125
@@
 	6600 3925 6750 3925
 $Comp
-L prius_gen2-rescue:R-Device R26
+L prius_gen2-rescue:R-Device-prius_gen2-rescue R26
 U 1 1 6121673C
 P 6600 3100
@@
 $EndComp
 $Comp
-L prius_gen2-rescue:+5V-power #PWR0136
+L prius_gen2-rescue:+5V-power-prius_gen2-rescue #PWR0136
 U 1 1 61216AB4
 P 6600 2825
@@
 	6575 4525 6750 4525
 $Comp
-L prius_gen2-rescue:GND-power #PWR0137
+L prius_gen2-rescue:GND-power-prius_gen2-rescue #PWR0137
 U 1 1 6121F68A
 P 5825 4500
@@
 $EndComp
 $Comp
-L prius_gen2-rescue:C-Device C19
+L prius_gen2-rescue:C-Device-prius_gen2-rescue C19
 U 1 1 6121FA1F
 P 5525 4250
@@
 $EndComp
 $Comp
-L prius_gen2-rescue:R-Device R25
+L prius_gen2-rescue:R-Device-prius_gen2-rescue R25
 U 1 1 61220142
 P 5825 4250
@@
 $EndComp
 $Comp
-L prius_gen2-rescue:R-Device R24
+L prius_gen2-rescue:R-Device-prius_gen2-rescue R24
 U 1 1 612205C1
 P 5825 3800
@@
 	5825 4450 5825 4500
 $Comp
-L prius_gen2-rescue:Conn_01x23-Connector_Generic J3
+L prius_gen2-rescue:Conn_01x23-Connector_Generic-prius_gen2-rescue J3
 U 1 1 60E8BF4D
 P 4175 4425
@@
 $EndComp
 $Comp
-L prius_gen2-rescue:Conn_01x14-Connector_Generic J4
+L prius_gen2-rescue:Conn_01x14-Connector_Generic-prius_gen2-rescue J4
 U 1 1 60E8DD9D
 P 8950 4125
@@
 $EndComp
 $Comp
-L prius_gen2-rescue:GND-power #PWR0138
+L prius_gen2-rescue:GND-power-prius_gen2-rescue #PWR0138
 U 1 1 60EB22A1
 P 8600 4990
@@
 	3975 3725 3725 3725
 $Comp
-L prius_gen2-rescue:+5V-power #PWR?
+L prius_gen2-rescue:+5V-power-prius_gen2-rescue #PWR?
 U 1 1 60F57711
 P 3725 5125
@@
 	3975 5025 3725 5025
 $Comp
-L prius_gen2-rescue:GND-power #PWR0187
+L prius_gen2-rescue:GND-power-prius_gen2-rescue #PWR0187
 U 1 1 61DA82E4
 P 7150 4850
