File: inputfilter.sch (KiCad schematic (older format))
At the start: 33 parts

Commit message: fixed schematics error
Parts:
- C43, C44, C45, C46, C47, C48, C49, C50, C51, C52: symbol prius_gen2-rescue:C-Device -> prius_gen2-rescue:C-Device-prius_gen2-rescue
- JP2, JP3: symbol prius_gen2-rescue:SolderJumper_2_Open-Jumper -> prius_gen2-rescue:SolderJumper_2_Open-Jumper-prius_gen2-rescue
- R41, R42, R43, R44, R45, R46, R47, R48, R49, R50, R51, R52, R53, R54, R55, R56, R57, R58, R60, R61: symbol prius_gen2-rescue:R-Device -> prius_gen2-rescue:R-Device-prius_gen2-rescue
- R59: value 510 -> 10k; symbol prius_gen2-rescue:R-Device -> prius_gen2-rescue:R-Device-prius_gen2-rescue
Changed lines of the file:
@@
 SIG_REV
 $Comp
-L prius_gen2-rescue:R-Device R46
+L prius_gen2-rescue:R-Device-prius_gen2-rescue R46
 U 1 1 61112451
 P 3650 1650
@@
 $EndComp
 $Comp
-L prius_gen2-rescue:R-Device R47
+L prius_gen2-rescue:R-Device-prius_gen2-rescue R47
 U 1 1 6111262B
 P 3650 1875
@@
 $EndComp
 $Comp
-L prius_gen2-rescue:R-Device R48
+L prius_gen2-rescue:R-Device-prius_gen2-rescue R48
 U 1 1 61112888
 P 3650 2100
@@
 $EndComp
 $Comp
-L prius_gen2-rescue:R-Device R49
+L prius_gen2-rescue:R-Device-prius_gen2-rescue R49
 U 1 1 61112A98
 P 3650 2325
@@
 $EndComp
 $Comp
-L prius_gen2-rescue:C-Device C45
+L prius_gen2-rescue:C-Device-prius_gen2-rescue C45
 U 1 1 61116E18
 P 4350 2750
@@
 $EndComp
 $Comp
-L prius_gen2-rescue:R-Device R50
+L prius_gen2-rescue:R-Device-prius_gen2-rescue R50
 U 1 1 6111700F
 P 4650 2750
@@
 $EndComp
 $Comp
-L prius_gen2-rescue:GND-power #PWR0175
+L prius_gen2-rescue:GND-power-prius_gen2-rescue #PWR0175
 U 1 1 61117506
 P 4275 3025
@@
 	4350 2975 4650 2975
 $Comp
-L prius_gen2-rescue:C-Device C46
+L prius_gen2-rescue:C-Device-prius_gen2-rescue C46
 U 1 1 61119644
 P 4975 2750
@@
 $EndComp
 $Comp
-L prius_gen2-rescue:R-Device R51
+L prius_gen2-rescue:R-Device-prius_gen2-rescue R51
 U 1 1 611196AE
 P 5275 2750
@@
 	4975 2975 5275 2975
 $Comp
-L prius_gen2-rescue:C-Device C47
+L prius_gen2-rescue:C-Device-prius_gen2-rescue C47
 U 1 1 6111BBB6
 P 5600 2750
@@
 $EndComp
 $Comp
-L prius_gen2-rescue:R-Device R52
+L prius_gen2-rescue:R-Device-prius_gen2-rescue R52
 U 1 1 6111BBBC
 P 5900 2750
@@
 	5600 2975 5900 2975
 $Comp
-L prius_gen2-rescue:C-Device C48
+L prius_gen2-rescue:C-Device-prius_gen2-rescue C48
 U 1 1 6111C8DF
 P 6225 2750
@@
 $EndComp
 $Comp
-L prius_gen2-rescue:R-Device R53
+L prius_gen2-rescue:R-Device-prius_gen2-rescue R53
 U 1 1 6111C8E5
 P 6525 2750
@@
 	6225 2975 6525 2975
 $Comp
-L prius_gen2-rescue:C-Device C49
+L prius_gen2-rescue:C-Device-prius_gen2-rescue C49
 U 1 1 6111D95E
 P 6850 2750
@@
 $EndComp
 $Comp
-L prius_gen2-rescue:R-Device R54
+L prius_gen2-rescue:R-Device-prius_gen2-rescue R54
 U 1 1 6111D964
 P 7150 2750
@@
 	3325 2325 3500 2325
 $Comp
-L prius_gen2-rescue:R-Device R45
+L prius_gen2-rescue:R-Device-prius_gen2-rescue R45
 U 1 1 61125FCC
 P 3650 1400
@@
 $EndComp
 $Comp
-L prius_gen2-rescue:+12V-power #PWR0176
+L prius_gen2-rescue:+12V-power-prius_gen2-rescue #PWR0176
 U 1 1 61126D64
 P 3200 1400
+AR Path="/61126D64" Ref="#PWR0176"  Part="1"
+AR Path="/610CA2CA/61126D64" Ref="#PWR0176"  Part="1"
 F 0 "#PWR0176" H 3200 1250 50  0001 C CNN
 F 1 "+12V" H 3215 1573 50  0000 C CNN
@@
 ENC_B
 $Comp
-L prius_gen2-rescue:R-Device R41
+L prius_gen2-rescue:R-Device-prius_gen2-rescue R41
 U 1 1 611359E8
 P 1475 4475
@@
 $EndComp
 $Comp
-L prius_gen2-rescue:R-Device R43
+L prius_gen2-rescue:R-Device-prius_gen2-rescue R43
 U 1 1 61135CED
 P 1925 4700
@@
 $EndComp
 $Comp
-L prius_gen2-rescue:SolderJumper_2_Open-Jumper JP2
+L prius_gen2-rescue:SolderJumper_2_Open-Jumper-prius_gen2-rescue JP2
 U 1 1 611364A8
 P 1475 4050
@@
 $EndComp
 $Comp
-L prius_gen2-rescue:+5V-power #PWR0177
+L prius_gen2-rescue:+5V-power-prius_gen2-rescue #PWR0177
 U 1 1 61136B01
 P 1475 3800
@@
 	2475 4700 2300 4700
 $Comp
-L prius_gen2-rescue:C-Device C43
+L prius_gen2-rescue:C-Device-prius_gen2-rescue C43
 U 1 1 6113A5DB
 P 2300 4900
@@
 $EndComp
 $Comp
-L prius_gen2-rescue:GND-power #PWR0178
+L prius_gen2-rescue:GND-power-prius_gen2-rescue #PWR0178
 U 1 1 6113AAEA
 P 2300 5125
@@
 ENC_A
 $Comp
-L prius_gen2-rescue:R-Device R42
+L prius_gen2-rescue:R-Device-prius_gen2-rescue R42
 U 1 1 6113ED6C
 P 1475 5950
@@
 $EndComp
 $Comp
-L prius_gen2-rescue:R-Device R44
+L prius_gen2-rescue:R-Device-prius_gen2-rescue R44
 U 1 1 6113ED72
 P 1925 6175
@@
 $EndComp
 $Comp
-L prius_gen2-rescue:SolderJumper_2_Open-Jumper JP3
+L prius_gen2-rescue:SolderJumper_2_Open-Jumper-prius_gen2-rescue JP3
 U 1 1 6113ED78
 P 1475 5525
@@
 $EndComp
 $Comp
-L prius_gen2-rescue:+5V-power #PWR0179
+L prius_gen2-rescue:+5V-power-prius_gen2-rescue #PWR0179
 U 1 1 6113ED7E
 P 1475 5275
@@
 	2475 6175 2300 6175
 $Comp
-L prius_gen2-rescue:C-Device C44
+L prius_gen2-rescue:C-Device-prius_gen2-rescue C44
 U 1 1 6113ED8C
 P 2300 6375
@@
 $EndComp
 $Comp
-L prius_gen2-rescue:GND-power #PWR0180
+L prius_gen2-rescue:GND-power-prius_gen2-rescue #PWR0180
 U 1 1 6113ED92
 P 2300 6600
@@
 MTEMP+
 $Comp
-L prius_gen2-rescue:R-Device R58
+L prius_gen2-rescue:R-Device-prius_gen2-rescue R58
 U 1 1 61157B0F
 P 9675 3425
@@
 $EndComp
 $Comp
-L prius_gen2-rescue:+5V-power #PWR0181
+L prius_gen2-rescue:+5V-power-prius_gen2-rescue #PWR0181
 U 1 1 61158191
 P 10050 3375
@@
 MTEMP-
 $Comp
-L prius_gen2-rescue:R-Device R59
+L prius_gen2-rescue:R-Device-prius_gen2-rescue R59
 U 1 1 6115C347
 P 9675 3750
-F 0 "R59" V 9882 3750 50  0000 C CNN
-F 1 "510" V 9791 3750 50  0000 C CNN
+F 0 "R59" V 9775 3850 50  0000 C CNN
+F 1 "10k" V 9775 3600 50  0000 C CNN
 F 2 "Resistor_SMD:R_0603_1608Metric" V 9605 3750 50  0001 C CNN
 F 3 "~" H 9675 3750 50  0001 C CNN
@@
 $EndComp
 $Comp
-L prius_gen2-rescue:R-Device R55
+L prius_gen2-rescue:R-Device-prius_gen2-rescue R55
 U 1 1 6115F0D1
 P 9450 3975
@@
 $EndComp
 $Comp
-L prius_gen2-rescue:C-Device C50
+L prius_gen2-rescue:C-Device-prius_gen2-rescue C50
 U 1 1 6115F539
 P 9900 3975
@@
 	9900 5925 9900 5825
 $Comp
-L prius_gen2-rescue:GND-power #PWR0183
+L prius_gen2-rescue:GND-power-prius_gen2-rescue #PWR0183
 U 1 1 6116D6AA
 P 9900 5925
@@
 $EndComp
 $Comp
-L prius_gen2-rescue:C-Device C52
+L prius_gen2-rescue:C-Device-prius_gen2-rescue C52
 U 1 1 6116D6A4
 P 9900 5675
@@
 $EndComp
 $Comp
-L prius_gen2-rescue:R-Device R57
+L prius_gen2-rescue:R-Device-prius_gen2-rescue R57
 U 1 1 6116D69E
 P 9450 5675
@@
 $EndComp
 $Comp
-L prius_gen2-rescue:R-Device R61
+L prius_gen2-rescue:R-Device-prius_gen2-rescue R61
 U 1 1 6116D698
 P 9675 5450
@@
 	9900 5075 9900 5025
 $Comp
-L prius_gen2-rescue:GND-power #PWR0184
+L prius_gen2-rescue:GND-power-prius_gen2-rescue #PWR0184
 U 1 1 61168C44
 P 9900 5075
@@
 $EndComp
 $Comp
-L prius_gen2-rescue:C-Device C51
+L prius_gen2-rescue:C-Device-prius_gen2-rescue C51
 U 1 1 61168C3E
 P 9900 4825
@@
 $EndComp
 $Comp
-L prius_gen2-rescue:R-Device R56
+L prius_gen2-rescue:R-Device-prius_gen2-rescue R56
 U 1 1 61168C38
 P 9450 4825
@@
 $EndComp
 $Comp
-L prius_gen2-rescue:R-Device R60
+L prius_gen2-rescue:R-Device-prius_gen2-rescue R60
 U 1 1 61168C32
 P 9675 4600
@@
 	9900 4175 9900 4225
 $Comp
-L prius_gen2-rescue:GND-power #PWR0182
+L prius_gen2-rescue:GND-power-prius_gen2-rescue #PWR0182
 U 1 1 6115F9E3
 P 9900 4225
