File: level_shifting.sch (KiCad schematic (older format))
At the start: 21 parts, among them U2 MCP602

Commit message: fixed schematics error
Parts:
- C14, C15, C16, C17: symbol prius_gen2-rescue:C-Device -> prius_gen2-rescue:C-Device-prius_gen2-rescue
- R10, R11, R12, R13, R14, R15, R16, R17, R18, R19, R20, R21, R6, R7, R8, R9: symbol prius_gen2-rescue:R-Device -> prius_gen2-rescue:R-Device-prius_gen2-rescue
- U2: symbol prius_gen2-rescue:MCP602-Amplifier_Operational -> prius_gen2-rescue:MCP602-Amplifier_Operational-prius_gen2-rescue
Changed lines of the file:
@@
 $EndDescr
 $Comp
-L prius_gen2-rescue:MCP602-Amplifier_Operational U?
+L prius_gen2-rescue:MCP602-Amplifier_Operational-prius_gen2-rescue U?
 U 1 1 6111F5BF
 P 5800 2550
@@
 $EndComp
 $Comp
-L prius_gen2-rescue:MCP602-Amplifier_Operational U?
+L prius_gen2-rescue:MCP602-Amplifier_Operational-prius_gen2-rescue U?
 U 2 1 6111F5C5
 P 5800 3825
@@
 $EndComp
 $Comp
-L prius_gen2-rescue:MCP602-Amplifier_Operational U?
+L prius_gen2-rescue:MCP602-Amplifier_Operational-prius_gen2-rescue U?
 U 3 1 6111F5CB
 P 7200 3575
@@
 $EndComp
 $Comp
-L prius_gen2-rescue:+5V-power #PWR?
+L prius_gen2-rescue:+5V-power-prius_gen2-rescue #PWR?
 U 1 1 6111F5D1
 P 7100 3200
@@
 $EndComp
 $Comp
-L prius_gen2-rescue:GND-power #PWR?
+L prius_gen2-rescue:GND-power-prius_gen2-rescue #PWR?
 U 1 1 6111F5D7
 P 7100 3975
@@
 	6400 3825 6150 3825
 $Comp
-L prius_gen2-rescue:R-Device R?
+L prius_gen2-rescue:R-Device-prius_gen2-rescue R?
 U 1 1 6111F5E3
 P 4775 2250
@@
 	4775 2450 5500 2450
 $Comp
-L prius_gen2-rescue:R-Device R?
+L prius_gen2-rescue:R-Device-prius_gen2-rescue R?
 U 1 1 6111F5EB
 P 4125 2400
@@
 $EndComp
 $Comp
-L prius_gen2-rescue:R-Device R?
+L prius_gen2-rescue:R-Device-prius_gen2-rescue R?
 U 1 1 6111F5F1
 P 4125 2700
@@
 	4425 2450 4425 2400
 $Comp
-L prius_gen2-rescue:C-Device C?
+L prius_gen2-rescue:C-Device-prius_gen2-rescue C?
 U 1 1 6111F5FD
 P 4425 2900
@@
 $EndComp
 $Comp
-L prius_gen2-rescue:GND-power #PWR?
+L prius_gen2-rescue:GND-power-prius_gen2-rescue #PWR?
 U 1 1 6111F603
 P 4425 3125
@@
 Connection ~ 4775 2450
 $Comp
-L prius_gen2-rescue:R-Device R?
+L prius_gen2-rescue:R-Device-prius_gen2-rescue R?
 U 1 1 6111F60D
 P 4775 2675
@@
 	4425 3075 4425 3050
 $Comp
-L prius_gen2-rescue:R-Device R?
+L prius_gen2-rescue:R-Device-prius_gen2-rescue R?
 U 1 1 6111F618
 P 5225 2875
@@
 	4775 2875 4775 2825
 $Comp
-L prius_gen2-rescue:R-Device R?
+L prius_gen2-rescue:R-Device-prius_gen2-rescue R?
 U 1 1 6111F624
 P 6150 2750
@@
 	5425 2950 5425 2875
 $Comp
-L prius_gen2-rescue:+5V-power #PWR?
+L prius_gen2-rescue:+5V-power-prius_gen2-rescue #PWR?
 U 1 1 6111F632
 P 4775 2050
@@
 	3975 2400 3750 2400
 $Comp
-L prius_gen2-rescue:R-Device R?
+L prius_gen2-rescue:R-Device-prius_gen2-rescue R?
 U 1 1 6111F63D
 P 6150 4050
@@
 $EndComp
 $Comp
-L prius_gen2-rescue:R-Device R?
+L prius_gen2-rescue:R-Device-prius_gen2-rescue R?
 U 1 1 6111F643
 P 5225 4150
@@
 $EndComp
 $Comp
-L prius_gen2-rescue:R-Device R?
+L prius_gen2-rescue:R-Device-prius_gen2-rescue R?
 U 1 1 6111F649
 P 4825 3925
@@
 $EndComp
 $Comp
-L prius_gen2-rescue:R-Device R?
+L prius_gen2-rescue:R-Device-prius_gen2-rescue R?
 U 1 1 6111F64F
 P 4825 3525
@@
 	4825 4075 4825 4150
 $Comp
-L prius_gen2-rescue:R-Device R?
+L prius_gen2-rescue:R-Device-prius_gen2-rescue R?
 U 1 1 6111F663
 P 4175 3675
@@
 $EndComp
 $Comp
-L prius_gen2-rescue:R-Device R?
+L prius_gen2-rescue:R-Device-prius_gen2-rescue R?
 U 1 1 6111F669
 P 4175 3975
@@
 	4475 3725 4475 3675
 $Comp
-L prius_gen2-rescue:C-Device C?
+L prius_gen2-rescue:C-Device-prius_gen2-rescue C?
 U 1 1 6111F675
 P 4475 4175
@@
 Connection ~ 4475 3975
 $Comp
-L prius_gen2-rescue:GND-power #PWR?
+L prius_gen2-rescue:GND-power-prius_gen2-rescue #PWR?
 U 1 1 6111F67D
 P 4475 4400
@@
 	4825 3725 4825 3775
 $Comp
-L prius_gen2-rescue:+5V-power #PWR?
+L prius_gen2-rescue:+5V-power-prius_gen2-rescue #PWR?
 U 1 1 6111F68C
 P 4825 3325
@@
 	4025 3675 3750 3675
 $Comp
-L prius_gen2-rescue:R-Device R?
+L prius_gen2-rescue:R-Device-prius_gen2-rescue R?
 U 1 1 6111F697
 P 3675 4950
@@
 $EndComp
 $Comp
-L prius_gen2-rescue:C-Device C?
+L prius_gen2-rescue:C-Device-prius_gen2-rescue C?
 U 1 1 6111F69D
 P 3950 5200
@@
 $EndComp
 $Comp
-L prius_gen2-rescue:R-Device R?
+L prius_gen2-rescue:R-Device-prius_gen2-rescue R?
 U 1 1 6111F6A3
 P 4300 5200
@@
 $EndComp
 $Comp
-L prius_gen2-rescue:GND-power #PWR?
+L prius_gen2-rescue:GND-power-prius_gen2-rescue #PWR?
 U 1 1 6111F6A9
 P 3950 5450
@@
 	3950 4950 4300 4950
 $Comp
-L prius_gen2-rescue:R-Device R?
+L prius_gen2-rescue:R-Device-prius_gen2-rescue R?
 U 1 1 6111F6BE
 P 5825 4925
@@
 $EndComp
 $Comp
-L prius_gen2-rescue:C-Device C?
+L prius_gen2-rescue:C-Device-prius_gen2-rescue C?
 U 1 1 6111F6C4
 P 6100 5175
@@
 $EndComp
 $Comp
-L prius_gen2-rescue:R-Device R?
+L prius_gen2-rescue:R-Device-prius_gen2-rescue R?
 U 1 1 6111F6CA
 P 6450 5175
@@
 $EndComp
 $Comp
-L prius_gen2-rescue:GND-power #PWR?
+L prius_gen2-rescue:GND-power-prius_gen2-rescue #PWR?
 U 1 1 6111F6D0
 P 6100 5425
