File: powersupply.sch (KiCad schematic (older format))
At the start: 20 parts, among them U7 LMR14020, U8 AZ1117-3.3

Commit message: fixed schematics error
Parts:
- C34, C36, C37, C38, C39, C40, C41, C42: symbol prius_gen2-rescue:C-Device -> prius_gen2-rescue:C-Device-prius_gen2-rescue
- C35: symbol prius_gen2-rescue:CP-Device -> prius_gen2-rescue:CP-Device-prius_gen2-rescue
- D4: symbol prius_gen2-rescue:ESD9B3.3ST5G-Diode -> prius_gen2-rescue:ESD9B3.3ST5G-Diode-prius_gen2-rescue
- D5, D6: symbol prius_gen2-rescue:D_Schottky-Device -> prius_gen2-rescue:D_Schottky-Device-prius_gen2-rescue
- L1, L2: symbol prius_gen2-rescue:INDUCTOR-pspice -> prius_gen2-rescue:INDUCTOR-pspice-prius_gen2-rescue
- R37, R38, R39, R40: symbol prius_gen2-rescue:R-Device -> prius_gen2-rescue:R-Device-prius_gen2-rescue
- U7: symbol prius_gen2-rescue:LMR14020-lmr14020 -> prius_gen2-rescue:LMR14020-lmr14020-prius_gen2-rescue
- U8: symbol prius_gen2-rescue:AZ1117-3.3-Regulator_Linear -> prius_gen2-rescue:AZ1117-3.3-Regulator_Linear-prius_gen2-rescue
Changed lines of the file:
@@
 $EndDescr
 $Comp
-L prius_gen2-rescue:AZ1117-3.3-Regulator_Linear U8
+L prius_gen2-rescue:AZ1117-3.3-Regulator_Linear-prius_gen2-rescue U8
 U 1 1 60E19B1F
 P 9250 3500
@@
 $EndComp
 $Comp
-L prius_gen2-rescue:D_Schottky-Device D5
+L prius_gen2-rescue:D_Schottky-Device-prius_gen2-rescue D5
 U 1 1 60E1C178
 P 2600 3250
@@
 $EndComp
 $Comp
-L prius_gen2-rescue:ESD9B3.3ST5G-Diode D4
+L prius_gen2-rescue:ESD9B3.3ST5G-Diode-prius_gen2-rescue D4
 U 1 1 60E1E16A
 P 2000 3500
@@
 $EndComp
 $Comp
-L prius_gen2-rescue:GND-power #PWR0159
+L prius_gen2-rescue:GND-power-prius_gen2-rescue #PWR0159
 U 1 1 60E1E77D
 P 2000 3800
@@
 $EndComp
 $Comp
-L prius_gen2-rescue:LMR14020-lmr14020 U7
+L prius_gen2-rescue:LMR14020-lmr14020-prius_gen2-rescue U7
 U 1 1 60E1F8E0
 P 5725 3450
@@
 $EndComp
 $Comp
-L prius_gen2-rescue:R-Device R37
+L prius_gen2-rescue:R-Device-prius_gen2-rescue R37
 U 1 1 60E21BB5
 P 3025 3450
@@
 $EndComp
 $Comp
-L prius_gen2-rescue:C-Device C34
+L prius_gen2-rescue:C-Device-prius_gen2-rescue C34
 U 1 1 60E2218B
 P 3025 3900
@@
 $EndComp
 $Comp
-L prius_gen2-rescue:INDUCTOR-pspice L1
+L prius_gen2-rescue:INDUCTOR-pspice-prius_gen2-rescue L1
 U 1 1 60E228C0
 P 3600 3250
@@
 $EndComp
 $Comp
-L prius_gen2-rescue:CP-Device C35
+L prius_gen2-rescue:CP-Device-prius_gen2-rescue C35
 U 1 1 60E23CAA
 P 4100 3525
@@
 $EndComp
 $Comp
-L prius_gen2-rescue:C-Device C36
+L prius_gen2-rescue:C-Device-prius_gen2-rescue C36
 U 1 1 60E24302
 P 4575 3525
@@
 	3850 3250 4100 3250
 $Comp
-L prius_gen2-rescue:GND-power #PWR0160
+L prius_gen2-rescue:GND-power-prius_gen2-rescue #PWR0160
 U 1 1 60E2C117
 P 3025 4150
@@
 $EndComp
 $Comp
-L prius_gen2-rescue:GND-power #PWR0161
+L prius_gen2-rescue:GND-power-prius_gen2-rescue #PWR0161
 U 1 1 60E2C381
 P 4100 3800
@@
 $EndComp
 $Comp
-L prius_gen2-rescue:GND-power #PWR0162
+L prius_gen2-rescue:GND-power-prius_gen2-rescue #PWR0162
 U 1 1 60E2C5C8
 P 4575 3800
@@
 	5050 3400 5050 3250
 $Comp
-L prius_gen2-rescue:R-Device R38
+L prius_gen2-rescue:R-Device-prius_gen2-rescue R38
 U 1 1 60E30342
 P 5025 3800
@@
 $EndComp
 $Comp
-L prius_gen2-rescue:GND-power #PWR0163
+L prius_gen2-rescue:GND-power-prius_gen2-rescue #PWR0163
 U 1 1 60E3058E
 P 5025 4050
@@
 	5025 3650 5025 3550
 $Comp
-L prius_gen2-rescue:C-Device C37
+L prius_gen2-rescue:C-Device-prius_gen2-rescue C37
 U 1 1 60E311D9
 P 5350 3975
@@
 $EndComp
 $Comp
-L prius_gen2-rescue:GND-power #PWR0164
+L prius_gen2-rescue:GND-power-prius_gen2-rescue #PWR0164
 U 1 1 60E316F6
 P 5350 4250
@@
 	5350 3825 5350 3750
 $Comp
-L prius_gen2-rescue:GND-power #PWR0165
+L prius_gen2-rescue:GND-power-prius_gen2-rescue #PWR0165
 U 1 1 60E327B6
 P 5825 4025
@@
 Connection ~ 5825 3975
 $Comp
-L prius_gen2-rescue:C-Device C38
+L prius_gen2-rescue:C-Device-prius_gen2-rescue C38
 U 1 1 60E384EC
 P 6525 3225
@@
 	6525 3000 6525 3075
 $Comp
-L prius_gen2-rescue:D_Schottky-Device D6
+L prius_gen2-rescue:D_Schottky-Device-prius_gen2-rescue D6
 U 1 1 60E3A3D8
 P 7050 3225
@@
 $EndComp
 $Comp
-L prius_gen2-rescue:INDUCTOR-pspice L2
+L prius_gen2-rescue:INDUCTOR-pspice-prius_gen2-rescue L2
 U 1 1 60E3ADD5
 P 7450 3500
@@
 	7050 3500 7200 3500
 $Comp
-L prius_gen2-rescue:GND-power #PWR0166
+L prius_gen2-rescue:GND-power-prius_gen2-rescue #PWR0166
 U 1 1 60E3CF68
 P 7050 3025
@@
 	7050 3025 7050 3075
 $Comp
-L prius_gen2-rescue:R-Device R39
+L prius_gen2-rescue:R-Device-prius_gen2-rescue R39
 U 1 1 60E417F0
 P 6400 3975
@@
 $EndComp
 $Comp
-L prius_gen2-rescue:R-Device R40
+L prius_gen2-rescue:R-Device-prius_gen2-rescue R40
 U 1 1 60E41BDB
 P 6900 3750
@@
 	6400 3750 6225 3750
 $Comp
-L prius_gen2-rescue:GND-power #PWR0167
+L prius_gen2-rescue:GND-power-prius_gen2-rescue #PWR0167
 U 1 1 60E4322F
 P 6400 4250
@@
 	6400 4250 6400 4125
 $Comp
-L prius_gen2-rescue:C-Device C39
+L prius_gen2-rescue:C-Device-prius_gen2-rescue C39
 U 1 1 60E4437D
 P 6900 4000
@@
 	6675 3750 6400 3750
 $Comp
-L prius_gen2-rescue:C-Device C40
+L prius_gen2-rescue:C-Device-prius_gen2-rescue C40
 U 1 1 60E4C1B8
 P 8125 3725
@@
 	7150 3750 7800 3750
 $Comp
-L prius_gen2-rescue:GND-power #PWR0168
+L prius_gen2-rescue:GND-power-prius_gen2-rescue #PWR0168
 U 1 1 60E4E5F9
 P 8125 3975
@@
 	8125 3975 8125 3875
 $Comp
-L prius_gen2-rescue:C-Device C41
+L prius_gen2-rescue:C-Device-prius_gen2-rescue C41
 U 1 1 60E50974
 P 8575 3725
@@
 $EndComp
 $Comp
-L prius_gen2-rescue:GND-power #PWR0169
+L prius_gen2-rescue:GND-power-prius_gen2-rescue #PWR0169
 U 1 1 60E5097A
 P 8575 3975
@@
 Connection ~ 8575 3500
 $Comp
-L prius_gen2-rescue:GND-power #PWR0170
+L prius_gen2-rescue:GND-power-prius_gen2-rescue #PWR0170
 U 1 1 60E55CFA
 P 9250 3975
@@
 	9250 3975 9250 3800
 $Comp
-L prius_gen2-rescue:+3V3-power #PWR0171
+L prius_gen2-rescue:+3V3-power-prius_gen2-rescue #PWR0171
 U 1 1 60E57207
 P 9875 3350
@@
 $EndComp
 $Comp
-L prius_gen2-rescue:GND-power #PWR0172
+L prius_gen2-rescue:GND-power-prius_gen2-rescue #PWR0172
 U 1 1 60E57682
 P 9875 3975
@@
 	9875 3575 9875 3500
 $Comp
-L prius_gen2-rescue:C-Device C42
+L prius_gen2-rescue:C-Device-prius_gen2-rescue C42
 U 1 1 60E57387
 P 9875 3725
@@
 	9875 3500 9875 3350
 $Comp
-L prius_gen2-rescue:PWR_FLAG-power #FLG0101
+L prius_gen2-rescue:PWR_FLAG-power-prius_gen2-rescue #FLG0101
 U 1 1 60E727E5
 P 2150 3250
@@
 	2150 3250 2450 3250
 $Comp
-L prius_gen2-rescue:PWR_FLAG-power #FLG0102
+L prius_gen2-rescue:PWR_FLAG-power-prius_gen2-rescue #FLG0102
 U 1 1 60E72D3D
 P 8125 3500
@@
 $EndComp
 $Comp
-L prius_gen2-rescue:+5V-power #PWR0173
+L prius_gen2-rescue:+5V-power-prius_gen2-rescue #PWR0173
 U 1 1 60E7481E
 P 8575 3350
@@
 	8575 3350 8575 3500
 $Comp
-L prius_gen2-rescue:+12V-power #PWR0174
+L prius_gen2-rescue:+12V-power-prius_gen2-rescue #PWR0174
 U 1 1 60FDA2CE
 P 1550 3150
+AR Path="/60FDA2CE" Ref="#PWR0174"  Part="1"
+AR Path="/60E19204/60FDA2CE" Ref="#PWR0174"  Part="1"
 F 0 "#PWR0174" H 1550 3000 50  0001 C CNN
 F 1 "+12V" H 1565 3323 50  0000 C CNN
@@
 Connection ~ 5050 3250
 $Comp
-L prius_gen2-rescue:PWR_FLAG-power #FLG0103
+L prius_gen2-rescue:PWR_FLAG-power-prius_gen2-rescue #FLG0103
 U 1 1 61AB96E0
 P 5250 3250
