File: prius_gen2.sch (KiCad schematic (older format))
At the start: 33 parts, among them J1 Conn_02x05_Odd_Even, J2 Conn_01x06, Q1 IRLZ14SPBF, Q2 IRLZ14SPBF, SW1 SW_Push, SW2 SW_Push, U9 STM32F103VBTx, Y1 8MHz

Commit message: fixed schematics error
Parts:
- C1, C12, C2: symbol prius_gen2-rescue:C-Device -> prius_gen2-rescue:C-Device-prius_gen2-rescue
- C10, C11, C3, C4, C5, C6, C7, C8, C9: symbol prius_gen2-rescue:C_Small-Device -> prius_gen2-rescue:C_Small-Device-prius_gen2-rescue
- D1, D7: symbol prius_gen2-rescue:LED-Device -> prius_gen2-rescue:LED-Device-prius_gen2-rescue
- FB1: symbol prius_gen2-rescue:Ferrite_Bead-Device -> prius_gen2-rescue:Ferrite_Bead-Device-prius_gen2-rescue
- J1: symbol prius_gen2-rescue:Conn_02x05_Odd_Even-Connector_Generic -> prius_gen2-rescue:Conn_02x05_Odd_Even-Connector_Generic-prius_gen2-rescue
- J2: symbol prius_gen2-rescue:Conn_01x06-Connector_Generic -> prius_gen2-rescue:Conn_01x06-Connector_Generic-prius_gen2-rescue
- Q1, Q2: symbol prius_gen2-rescue:IRLZ34N-Transistor_FET -> prius_gen2-rescue:IRLZ34N-Transistor_FET-prius_gen2-rescue
- R1, R2, R3, R4, R5, R62, R63, R64: symbol prius_gen2-rescue:R-Device -> prius_gen2-rescue:R-Device-prius_gen2-rescue
- SW1, SW2: symbol prius_gen2-rescue:SW_Push-Switch -> prius_gen2-rescue:SW_Push-Switch-prius_gen2-rescue
- TP1, TP2: symbol prius_gen2-rescue:TestPoint-Connector -> prius_gen2-rescue:TestPoint-Connector-prius_gen2-rescue
- U9: symbol prius_gen2-rescue:STM32F103VBTx-MCU_ST_STM32F1 -> prius_gen2-rescue:STM32F103VBTx-MCU_ST_STM32F1-prius_gen2-rescue
- Y1: symbol prius_gen2-rescue:Crystal-Device -> prius_gen2-rescue:Crystal-Device-prius_gen2-rescue
Connections:
- wire segments 231 -> 241
Other:
- moved on the sheet: C1, C10, C11, C12, C2, C3, C4, C5, C6, C7, C8, C9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

Commit message: updated silk and manuf. files
Parts:
- removed TP1, TP2: TestPoint, TestPoint:TestPoint_Pad_1.5x1.5mm, symbol prius_gen2-rescue:TestPoint-Connector-prius_gen2-rescue
Connections:
- wire segments 241 -> 237
Changed lines of the file:
@@
 	14215 4770 14665 4770
-$Comp
-L prius_gen2-rescue:TestPoint-Connector-prius_gen2-rescue TP1
-U 1 1 60FD29FA
-P 11715 7645
-F 0 "TP1" H 11773 7763 50  0000 L CNN
-F 1 "TestPoint" H 11773 7672 50  0000 L CNN
-F 2 "TestPoint:TestPoint_Pad_1.5x1.5mm" H 11915 7645 50  0001 C CNN
-F 3 "~" H 11915 7645 50  0001 C CNN
-	1    11715 7645
-	1    0    0    -1
-$EndComp
-$Comp
-L prius_gen2-rescue:TestPoint-Connector-prius_gen2-rescue TP2
-U 1 1 60FD7C7A
-P 11715 8045
-F 0 "TP2" H 11773 8163 50  0000 L CNN
-F 1 "TestPoint" H 11773 8072 50  0000 L CNN
-F 2 "TestPoint:TestPoint_Pad_1.5x1.5mm" H 11915 8045 50  0001 C CNN
-F 3 "~" H 11915 8045 50  0001 C CNN
-	1    11715 8045
-	1    0    0    -1
-$EndComp
-Text Label 12140 7770 2    50   ~ 0
-UART3_TX
-Wire Wire Line
-	12140 7770 11715 7770
-Wire Wire Line
-	11715 7770 11715 7645
-Text Label 12115 8195 2    50   ~ 0
-UART3_RX
-Wire Wire Line
-	12115 8195 11715 8195
-Wire Wire Line
-	11715 8195 11715 8045
 $Comp
 L prius_gen2-rescue:+3V3-power-prius_gen2-rescue #PWR01
