File: prius_gen2.kicad_pcb (KiCad board)
At the start: 4 copper layers, 130.6 x 65 mm, 138 parts, among them J1 Conn_02x05_Odd_Even, J2 Conn_01x06, J3 Conn_01x23, J4 Conn_01x14, Q1 Q_NPN_BEC, Q2 Q_PNP_BEC, Q3 Q_NPN_BEC, Q4 Q_PNP_BEC, SW1 SW_Push, SW2 SW_Push, U1 STM32F407VETx, U2 ULN2003A, U3 AD2S1205YSTZ, U4 TJA1051T-3, U5 LMR14020, U6 AZ1117-3.3, U7 MCP602, U8 AD8676xR, Y1 8MHz, Y2 8.192MHz

Commit message: added USB
Parts:
- added C16: 100n, Capacitor_SMD:C_0603_1608Metric, F.Cu at (182.4, 96.8)
- added D11: schottky, Diode_SMD:D_SOD-123, F.Cu at (175.5, 86.1)
- added J5: ~, Connector_PinSocket_2.54mm:PinSocket_1x05_P2.54mm_Vertical, F.Cu at (179.5, 87.5)
- added R14: 100k, Resistor_SMD:R_0402_1005Metric, F.Cu at (182.4, 99.5)
- added U9: ~, Package_TO_SOT_SMD:SOT-23-6, F.Cu at (175.2, 91.5)
- R24, R51: value R -> 17.4k
- renumbered CH1N to TP1, CH2N to TP2, CH3N to TP3, CH3 to TP4, CH2 to TP5, CH1 to TP6, BKIN to TP7
Connections:
- U1 pad 70: /CAN_RX -> /USB_D-
- U1 pad 71: /CAN_TX -> /USB_D+
- U1 pad 95: unconnected-(U1-Pad95) -> /CAN_RX
- U1 pad 96: unconnected-(U1-Pad96) -> /CAN_TX
Routing:
- net /USB_D-: track 0.00 -> 34.6 mm, vias 0 -> 2
- net /USB_D+: track 0.00 -> 33.7 mm, vias 0 -> 2
- net +5V: track 245.3 -> 265.2 mm, vias 11 -> 12
- net Net-(D11-Pad2): track 0.00 -> 9.10 mm, vias 0 -> 2
- net /CAN_TX: track 41.6 -> 49.9 mm, vias 0 -> 2
- net /CAN_RX: track 38.6 -> 45.2 mm
- net USB_SHIELD: track 0.00 -> 4.27 mm
Other:
- board text added: "Designed in Los Angeles github.com/ksmola/PriusG2"
- board text removed: "github.com/ksmola/PriusG2"
