File: communication.kicad_sch (KiCad schematic)
At the start: 17 parts, among them J5 Conn_01x03_Male, SW3 RESET, SW4 BOOT, U5 TJA1051T-3, U6 ESP32-WROOM-32

Commit message: started adding AD2S
Parts:
- removed C30, C31, C33: .1u, Capacitor_SMD:C_0603_1608Metric, symbol prius_gen2-rescue:C-Device-prius_gen2-rescue
- removed C32: 10u, Capacitor_SMD:C_0603_1608Metric, symbol prius_gen2-rescue:C-Device-prius_gen2-rescue
- removed D3: LED, LED_SMD:LED_0603_1608Metric_Castellated, symbol prius_gen2-rescue:LED-Device-prius_gen2-rescue
- removed J5: Conn_01x03_Male, Connector_PinSocket_1.27mm:PinSocket_1x03_P1.27mm_Vertical_SMD_Pin1Left, symbol prius_gen2-rescue:Conn_01x03_Male-Connector-prius_gen2-rescue
- removed R34, R36: 10k, Resistor_SMD:R_0603_1608Metric, symbol prius_gen2-rescue:R-Device-prius_gen2-rescue
- removed R35: 1k, Resistor_SMD:R_0603_1608Metric, symbol prius_gen2-rescue:R-Device-prius_gen2-rescue
- removed SW3: RESET, Button_Switch_SMD:SW_SPST_EVQQ2, symbol prius_gen2-rescue:SW_Push-Switch-prius_gen2-rescue
- removed SW4: BOOT, Button_Switch_SMD:SW_SPST_EVQQ2, symbol prius_gen2-rescue:SW_Push-Switch-prius_gen2-rescue
- removed U6: ESP32-WROOM-32, RF_Module:ESP32-WROOM-32, symbol prius_gen2-rescue:ESP32-WROOM-32-RF_Module-prius_gen2-rescue
- C28: renamed from C?; value (none) -> 100nF; footprint (none) -> Capacitor_SMD:C_0603_1608Metric
- R25: renamed from R33; symbol prius_gen2-rescue:R-Device-prius_gen2-rescue -> Device:R
- renumbered D2 to D3, JP1 to JP3, U5 to U4
Connections:
- no-connect marks 26 -> 0
Other:
- note removed: "ESP32 WiFi interface"
- note removed: "Programming port"
- moved on the sheet: C28, D3, JP3, R25, U4
