File: inputfilter.kicad_sch (KiCad schematic)
At the start: 33 parts

Commit message: started adding AD2S
Parts:
- removed C45, C46, C47, C48, C49, C51, C52: 1u, Capacitor_SMD:C_0603_1608Metric, symbol prius_gen2-rescue:C-Device-prius_gen2-rescue
- removed R45: 4.7k, Resistor_SMD:R_0603_1608Metric, symbol prius_gen2-rescue:R-Device-prius_gen2-rescue
- removed R46, R47, R48, R49: 3.3k, Resistor_SMD:R_0603_1608Metric, symbol prius_gen2-rescue:R-Device-prius_gen2-rescue
- removed R50, R51, R52, R53, R54: 1.2k, Resistor_SMD:R_0603_1608Metric, symbol prius_gen2-rescue:R-Device-prius_gen2-rescue
- removed R56, R57, R60, R61: 10k, Resistor_SMD:R_0603_1608Metric, symbol prius_gen2-rescue:R-Device-prius_gen2-rescue
- C13: renamed from C43; symbol prius_gen2-rescue:C-Device-prius_gen2-rescue -> Device:C
- C14: renamed from C44; symbol prius_gen2-rescue:C-Device-prius_gen2-rescue -> Device:C
- C15: renamed from C50; symbol prius_gen2-rescue:C-Device-prius_gen2-rescue -> Device:C
- R10: renamed from R44; symbol prius_gen2-rescue:R-Device-prius_gen2-rescue -> Device:R
- R11: renamed from R55; symbol prius_gen2-rescue:R-Device-prius_gen2-rescue -> Device:R
- R12: renamed from R58; symbol prius_gen2-rescue:R-Device-prius_gen2-rescue -> Device:R
- R13: renamed from R59; symbol prius_gen2-rescue:R-Device-prius_gen2-rescue -> Device:R
- R7: renamed from R41; symbol prius_gen2-rescue:R-Device-prius_gen2-rescue -> Device:R
- R8: renamed from R42; symbol prius_gen2-rescue:R-Device-prius_gen2-rescue -> Device:R
- R9: renamed from R43; symbol prius_gen2-rescue:R-Device-prius_gen2-rescue -> Device:R
- renumbered JP2 to JP1, JP3 to JP2
Other:
- moved on the sheet: C13, C14, C15, JP1, JP2, R10, R11, R12, R13, R7, R8, R9

Commit message: routed ad2s
Parts:
- R10, R13, R9: LCSC (none) -> C25804
Changed lines of the file:
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@@
+      (effects (font (size 1.27 1.27)) hide)
+    )
+    (property "LCSC" "C25804" (id 4) (at 121.92 83.82 90)
       (effects (font (size 1.27 1.27)) hide)
     )
@@
       (effects (font (size 1.27 1.27)) hide)
     )
+    (property "LCSC" "C25804" (id 4) (at 121.92 121.285 90)
+      (effects (font (size 1.27 1.27)) hide)
+    )
     (pin "1")
     (pin "2")
@@
       (effects (font (size 1.27 1.27)) hide)
     )
+    (property "LCSC" "C25804" (id 4) (at 187.325 96.52 90)
+      (effects (font (size 1.27 1.27)) hide)
+    )
