File: level_shifting.kicad_sch (KiCad schematic)
At the start: 23 parts

Commit message: started adding AD2S
Parts:
- C38, C41: renamed from C?; value (none) -> 1u; footprint (none) -> Capacitor_SMD:C_0603_1608Metric; symbol prius_gen2-rescue:C-Device-prius_gen2-rescue -> Device:C
- C39, C40: renamed from C?; value (none) -> 1n; footprint (none) -> Capacitor_SMD:C_0603_1608Metric; symbol prius_gen2-rescue:C-Device-prius_gen2-rescue -> Device:C
- R30, R35, R42, R43, R44, R45: renamed from R?; value (none) -> 10K; footprint (none) -> Resistor_SMD:R_0603_1608Metric; symbol prius_gen2-rescue:R-Device-prius_gen2-rescue -> Device:R
- R31, R32, R33, R34, R40, R41: renamed from R?; value (none) -> 100K; footprint (none) -> Resistor_SMD:R_0603_1608Metric; symbol prius_gen2-rescue:R-Device-prius_gen2-rescue -> Device:R
- R36, R38: renamed from R?; value (none) -> 33K; footprint (none) -> Resistor_SMD:R_0603_1608Metric; symbol prius_gen2-rescue:R-Device-prius_gen2-rescue -> Device:R
- R37, R39: renamed from R?; value (none) -> 15K; footprint (none) -> Resistor_SMD:R_0603_1608Metric; symbol prius_gen2-rescue:R-Device-prius_gen2-rescue -> Device:R
- U7: renamed from U?; value (none) -> MCP602; footprint (none) -> Package_SO:SOIC-8-1EP_3.9x4.9mm_P1.27mm_EP2.29x3mm

Commit message: routed ad2s
Parts:
- R30, R35, R42, R45: LCSC (none) -> C25804
Changed lines of the file:
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@@
+      (effects (font (size 1.27 1.27)) hide)
+    )
+    (property "LCSC" "C25804" (id 4) (at 93.345 125.73 90)
       (effects (font (size 1.27 1.27)) hide)
     )
@@
       (effects (font (size 1.27 1.27)) hide)
     )
+    (property "LCSC" "C25804" (id 4) (at 109.22 132.08 0)
+      (effects (font (size 1.27 1.27)) hide)
+    )
     (pin "1")
     (pin "2")
@@
     )
     (property "Datasheet" "~" (id 3) (at 147.955 125.095 0)
+      (effects (font (size 1.27 1.27)) hide)
+    )
+    (property "LCSC" "C25804" (id 4) (at 147.955 125.095 90)
       (effects (font (size 1.27 1.27)) hide)
     )
@@
       (effects (font (size 1.27 1.27)) hide)
     )
+    (property "LCSC" "C25804" (id 4) (at 163.83 131.445 0)
+      (effects (font (size 1.27 1.27)) hide)
+    )
