File: powersupply.kicad_sch (KiCad schematic)
At the start: 20 parts, among them U7 LMR14020, U8 AZ1117-3.3

Commit message: started adding AD2S
Parts:
- C29: renamed from C34; symbol prius_gen2-rescue:C-Device-prius_gen2-rescue -> Device:C
- C31: renamed from C36; symbol prius_gen2-rescue:C-Device-prius_gen2-rescue -> Device:C
- C32: renamed from C37; symbol prius_gen2-rescue:C-Device-prius_gen2-rescue -> Device:C
- C33: renamed from C38; symbol prius_gen2-rescue:C-Device-prius_gen2-rescue -> Device:C
- C34: renamed from C39; symbol prius_gen2-rescue:C-Device-prius_gen2-rescue -> Device:C
- C35: renamed from C40; symbol prius_gen2-rescue:C-Device-prius_gen2-rescue -> Device:C
- C36: renamed from C41; symbol prius_gen2-rescue:C-Device-prius_gen2-rescue -> Device:C
- C37: renamed from C42; symbol prius_gen2-rescue:C-Device-prius_gen2-rescue -> Device:C
- R26: renamed from R37; symbol prius_gen2-rescue:R-Device-prius_gen2-rescue -> Device:R
- R27: renamed from R38; symbol prius_gen2-rescue:R-Device-prius_gen2-rescue -> Device:R
- R28: renamed from R39; symbol prius_gen2-rescue:R-Device-prius_gen2-rescue -> Device:R
- R29: renamed from R40; symbol prius_gen2-rescue:R-Device-prius_gen2-rescue -> Device:R
- renumbered C35 to C30, U7 to U5, U8 to U6

Commit message: routed ad2s
Parts:
- C32: LCSC (none) -> C302008
- R27: LCSC (none) -> C25804
- R29: LCSC (none) -> C23231
Changed lines of the file:
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@@
+      (effects (font (size 1.27 1.27)) hide)
+    )
+    (property "LCSC" "C25804" (id 4) (at 127.635 96.52 0)
       (effects (font (size 1.27 1.27)) hide)
     )
@@
     )
     (property "Datasheet" "~" (id 3) (at 135.89 100.965 0)
+      (effects (font (size 1.27 1.27)) hide)
+    )
+    (property "LCSC" "C302008" (id 4) (at 135.89 100.965 0)
       (effects (font (size 1.27 1.27)) hide)
     )
@@
       (effects (font (size 1.27 1.27)) hide)
     )
+    (property "LCSC" "C23231" (id 4) (at 175.26 95.25 90)
+      (effects (font (size 1.27 1.27)) hide)
+    )

Commit message: v0.5 production files
Changed lines of the file:
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@@
       (effects (font (size 1.27 1.27)) (justify right))
     )
-    (property "Value" "D_Schottky" (at 181.102 83.058 90)
+    (property "Value" "D_Schottky" (at 189.23 74.295 90)
       (effects (font (size 1.27 1.27)) (justify right))
     )
