File: prius_gen2.kicad_sch (KiCad schematic)
At the start: 41 parts, among them J2 Conn_01x06, SW1 SW_Push, SW2 SW_Push, U1 STM32F407VETx, Y1 8MHz

Commit message: v0.5 production files
Parts:
- removed TP2: TestPoint, TestPoint:TestPoint_Keystone_5000-5004_Miniature, symbol Connector:TestPoint
Connections:
- net TIM1_BKIN: now also U1.66 (PC9)
- net ADC12 renamed ADC123_IN10
- net ADC13 renamed ADC123_IN11
- net ADC14 renamed ADC123_IN12
- net ADC5 renamed ADC123_IN1
- net ADC8 renamed ADC123_IN2
- net TIM1_CH2N: no longer names the net of U1.53 (PB14)
- net TIM3_ETR: no longer names the net of U1.83 (PD2)
- no-connect marks 52 -> 53
Other:
- note removed: "ADC123_IN1"
- note removed: "ADC123_IN10"
- note removed: "ADC123_IN11"
- note removed: "ADC123_IN12"
- note removed: "ADC123_IN2"
Changed lines of the file:
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@@
   (no_connect (at 196.85 196.85))
   (no_connect (at 151.13 153.67))
+  (no_connect (at 151.13 191.77))
   (no_connect (at 196.85 100.33))
   (no_connect (at 151.13 148.59))
@@
   (no_connect (at 151.13 151.13))
   (no_connect (at 196.85 146.05))
-  (no_connect (at 196.85 209.55))
   (no_connect (at 151.13 201.93))
   (no_connect (at 151.13 212.09))
   (no_connect (at 151.13 222.25))
   (no_connect (at 196.85 151.13))
+  (no_connect (at 196.85 179.07))
   (no_connect (at 151.13 194.31))
   (no_connect (at 196.85 153.67))
@@
     (stroke (width 0) (type default))
   )
-  (wire (pts (xy 368.3 140.97) (xy 374.65 140.97))
+  (wire (pts (xy 368.3 140.97) (xy 382.27 140.97))
+    (stroke (width 0) (type default))
+  )
+  (wire (pts (xy 196.85 209.55) (xy 207.01 209.55))
     (stroke (width 0) (type default))
   )
@@
     (stroke (width 0) (type default))
   )
-  (wire (pts (xy 196.85 105.41) (xy 205.105 105.41))
+  (wire (pts (xy 196.85 105.41) (xy 208.915 105.41))
     (stroke (width 0) (type default))
   )
@@
     (stroke (width 0) (type default))
   )
-  (wire (pts (xy 196.85 102.87) (xy 205.105 102.87))
+  (wire (pts (xy 196.85 102.87) (xy 208.915 102.87))
     (stroke (width 0) (type default))
   )
@@
     (stroke (width 0) (type default))
   )
-  (wire (pts (xy 196.85 186.69) (xy 207.01 186.69))
+  (wire (pts (xy 196.85 186.69) (xy 208.915 186.69))
     (stroke (width 0) (type default))
   )
@@
     (stroke (width 0) (type default))
   )
-  (wire (pts (xy 208.28 179.07) (xy 196.85 179.07))
-    (stroke (width 0) (type default))
-  )
   (wire (pts (xy 327.66 148.59) (xy 322.58 148.59))
     (stroke (width 0) (type default))
@@
     (stroke (width 0) (type default))
   )
-  (wire (pts (xy 374.65 146.05) (xy 368.3 146.05))
+  (wire (pts (xy 382.27 146.05) (xy 368.3 146.05))
     (stroke (width 0) (type default))
   )
@@
     (stroke (width 0) (type default))
   )
-  (wire (pts (xy 337.82 151.13) (xy 346.71 151.13))
+  (wire (pts (xy 333.375 151.13) (xy 346.71 151.13))
     (stroke (width 0) (type default))
   )
@@
     (stroke (width 0) (type default))
   )
-  (wire (pts (xy 346.71 148.59) (xy 337.82 148.59))
+  (wire (pts (xy 346.71 148.59) (xy 333.375 148.59))
     (stroke (width 0) (type default))
   )
@@
     (stroke (width 0) (type default))
   )
-  (wire (pts (xy 207.01 191.77) (xy 196.85 191.77))
+  (wire (pts (xy 208.915 191.77) (xy 196.85 191.77))
     (stroke (width 0) (type default))
   )
@@
     (stroke (width 0) (type default))
   )
-  (wire (pts (xy 151.13 191.77) (xy 140.97 191.77))
-    (stroke (width 0) (type default))
-  )
   (wire (pts (xy 68.326 200.406) (xy 68.326 202.946))
     (stroke (width 0) (type default))
@@
     (stroke (width 0) (type default))
   )
-  (wire (pts (xy 207.01 189.23) (xy 196.85 189.23))
+  (wire (pts (xy 208.915 189.23) (xy 196.85 189.23))
     (stroke (width 0) (type default))
   )
@@
     (effects (font (size 1.27 1.27)) (justify left bottom))
   )
-  (text "ADC123_IN2" (at 207.645 105.41 0)
-    (effects (font (size 1.27 1.27)) (justify left bottom))
-  )
   (text "ok" (at 209.55 115.57 0)
     (effects (font (size 1.27 1.27)) (justify left bottom))
@@
     (effects (font (size 1.27 1.27)) (justify left bottom))
   )
-  (text "ADC123_IN11" (at 208.28 189.23 0)
-    (effects (font (size 1.27 1.27)) (justify left bottom))
-  )
-  (text "ADC123_IN1" (at 207.645 102.87 0)
-    (effects (font (size 1.27 1.27)) (justify left bottom))
-  )
   (text "ok" (at 209.55 117.475 0)
     (effects (font (size 1.27 1.27)) (justify left bottom))
@@
     (effects (font (size 1.27 1.27)) (justify left bottom))
   )
-  (text "ADC123_IN10" (at 208.28 186.69 0)
-    (effects (font (size 1.27 1.27)) (justify left bottom))
-  )
-  (text "ADC123_IN12" (at 208.28 191.77 0)
-    (effects (font (size 1.27 1.27)) (justify left bottom))
-  )
   (text "SWD DEBUG" (at 239.776 239.268 0)
     (effects (font (size 1.27 1.27)) (justify left bottom))
@@
     (effects (font (size 1.27 1.27)) (justify left bottom))
   )
-  (label "ADC12" (at 39.37 238.76 0) (fields_autoplaced)
+  (label "ADC123_IN10" (at 39.37 238.76 0) (fields_autoplaced)
     (effects (font (size 1.27 1.27)) (justify left bottom))
   )
@@
     (effects (font (size 1.27 1.27)) (justify right bottom))
   )
-  (label "ADC5" (at 337.82 148.59 0) (fields_autoplaced)
+  (label "ADC123_IN1" (at 333.375 148.59 0) (fields_autoplaced)
     (effects (font (size 1.27 1.27)) (justify left bottom))
   )
@@
     (effects (font (size 1.27 1.27)) (justify right bottom))
   )
-  (label "ADC14" (at 207.01 191.77 180) (fields_autoplaced)
-    (effects (font (size 1.27 1.27)) (justify right bottom))
-  )
-  (label "ADC8" (at 205.105 105.41 180) (fields_autoplaced)
+  (label "ADC123_IN12" (at 208.915 191.77 180) (fields_autoplaced)
+    (effects (font (size 1.27 1.27)) (justify right bottom))
+  )
+  (label "ADC123_IN2" (at 208.915 105.41 180) (fields_autoplaced)
     (effects (font (size 1.27 1.27)) (justify right bottom))
   )
@@
     (effects (font (size 1.27 1.27)) (justify right bottom))
   )
+  (label "TIM1_BKIN" (at 207.01 209.55 180) (fields_autoplaced)
+    (effects (font (size 1.27 1.27)) (justify right bottom))
+  )
   (label "~{CS}" (at 208.28 158.75 180) (fields_autoplaced)
     (effects (font (size 1.27 1.27)) (justify right bottom))
   )
-  (label "TIM3_ETR" (at 140.97 191.77 0) (fields_autoplaced)
-    (effects (font (size 1.27 1.27)) (justify left bottom))
-  )
   (label "EXC-" (at 281.94 130.81 0) (fields_autoplaced)
     (effects (font (size 1.27 1.27)) (justify left bottom))
@@
     (effects (font (size 1.27 1.27)) (justify left bottom))
   )
-  (label "ADC13" (at 207.01 189.23 180) (fields_autoplaced)
-    (effects (font (size 1.27 1.27)) (justify right bottom))
-  )
-  (label "ADC14" (at 374.65 140.97 180) (fields_autoplaced)
-    (effects (font (size 1.27 1.27)) (justify right bottom))
-  )
-  (label "TIM1_CH2N" (at 208.28 179.07 180) (fields_autoplaced)
+  (label "ADC123_IN11" (at 208.915 189.23 180) (fields_autoplaced)
+    (effects (font (size 1.27 1.27)) (justify right bottom))
+  )
+  (label "ADC123_IN12" (at 382.27 140.97 180) (fields_autoplaced)
     (effects (font (size 1.27 1.27)) (justify right bottom))
   )
@@
     (effects (font (size 1.27 1.27)) (justify left bottom))
   )
-  (label "ADC8" (at 337.82 151.13 0) (fields_autoplaced)
+  (label "ADC123_IN2" (at 333.375 151.13 0) (fields_autoplaced)
     (effects (font (size 1.27 1.27)) (justify left bottom))
   )
@@
     (effects (font (size 1.27 1.27)) (justify right bottom))
   )
-  (label "ADC13" (at 374.65 146.05 180) (fields_autoplaced)
+  (label "ADC123_IN11" (at 382.27 146.05 180) (fields_autoplaced)
     (effects (font (size 1.27 1.27)) (justify right bottom))
   )
@@
     (effects (font (size 1.27 1.27)) (justify right bottom))
   )
-  (label "ADC12" (at 207.01 186.69 180) (fields_autoplaced)
+  (label "ADC123_IN10" (at 208.915 186.69 180) (fields_autoplaced)
     (effects (font (size 1.27 1.27)) (justify right bottom))
   )
@@
     (effects (font (size 1.27 1.27)) (justify right bottom))
   )
-  (label "ADC5" (at 205.105 102.87 180) (fields_autoplaced)
+  (label "ADC123_IN1" (at 208.915 102.87 180) (fields_autoplaced)
     (effects (font (size 1.27 1.27)) (justify right bottom))
   )
@@
         )
       )
-    )
-  )
-  (symbol (lib_id "Connector:TestPoint") (at 208.28 179.07 270) (unit 1)
-    (in_bom yes) (on_board yes) (dnp no) (fields_autoplaced)
-    (property "Reference" "TP2" (at 213.36 179.0699 90)
-      (effects (font (size 1.27 1.27)) (justify left))
-    )
-    (property "Value" "TestPoint" (at 213.36 180.3399 90)
-      (effects (font (size 1.27 1.27)) (justify left) hide)
-    )
-    (property "Footprint" "TestPoint:TestPoint_Keystone_5000-5004_Miniature" (at 208.28 184.15 0)
-      (effects (font (size 1.27 1.27)) hide)
-    )
-    (property "Datasheet" "~" (at 208.28 184.15 0)
-      (effects (font (size 1.27 1.27)) hide)
-    )
-    (property "LCSC" "C238124" (at 208.28 179.07 90)
-      (effects (font (size 1.27 1.27)) hide)
-    )
-    (pin "1")
-    (instances
-      (project "prius_gen2"
-        (path "/1c27b0ef-4199-489c-80da-fdf964569958"
-          (reference "TP2") (unit 1)
-        )
-      )
